File: KiCAD/Pico_energymeter.kicad_sch (KiCad schematic)
At the start: 27 parts, among them J1 Conn_01x02_Pin, J2 Conn_01x03_Socket, J3 Conn_01x04_Pin, J4 Screw_Terminal_01x02, U1 Pico, U2 LM358, U3 HLK-PM01

Commit message: correct schematic
Parts:
- R12: value 10K -> 15K
Changed lines of the file:
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@@
 			)
 		)
-		(property "Value" "10K"
+		(property "Value" "15K"
 			(at 207.01 195.58 90)
 			(effects
